File: hw/DeutschlandLaenderStatus-r0.1/kicad-src/DeutschlandLaenderStatus.kicad_pcb (KiCad board)
At the start: 4 copper layers, 130 x 160 mm, 106 parts, among them J1 USB_C, SW1 SW_Push, SW2 SW_Push, SW3 SW_Push, U1 USBLC6-2, U10 SN74LVC2T45DCUR, U2 ESP32-S2, U3 TLV62569DRL, U4 LY68L6400SLIT, U5 W25Q128JVS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

Commit message: initial artwork created
Parts:
- added Ref**: Val**, kt-footprints:de-02 smoothed, F.Cu at (93.3, 94.2)
Routing:
- added copper zone on F.Cu, net GND
Other:
- board size 130 x 160 mm -> 117.7 x 147.4 mm
