File: hw/DeutschlandLaenderStatus-r0.1/kicad-src/DeutschlandLaenderStatus.kicad_pcb (KiCad board)
At the start: 4 copper layers, 109.8 x 145 mm, 108 parts, among them J1 USB_C, SW1 SW_Push, SW2 SW_Push, SW3 SW_Push, U1 USBLC6-2, U10 SN74LVC2T45DCUR, U2 ESP32-S2, U3 TLV62569DRL, U4 LY68L6400SLIT, U5 W25Q128JVS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

Commit message: PCB note updates
Routing:
- net /I2C_SCL: track 57.7 -> 42.5 mm, vias 3 -> 0
- net Net-(U7-Pad6): track 31.6 -> 36.9 mm, vias 2 -> 3
- net /USB_P: track 37.3 -> 39.6 mm
- net /USB_N: track 37.8 -> 39.9 mm
- net Net-(U7-Pad7): track 50.1 -> 48.1 mm, vias 2 -> 4
- net Net-(U6-Pad9): track 42.6 -> 44.5 mm
- net Net-(U6-Pad1): track 21.8 -> 20.4 mm
- net /SEG_IRQ: track 53.3 -> 54.6 mm, vias 3 -> 0
- net Net-(U6-Pad4): track 20.2 -> 21.4 mm
- net Net-(U6-Pad5): track 20.9 -> 21.9 mm
- net Net-(C4-Pad1): track 16.5 -> 15.6 mm
- net Net-(U6-Pad2): track 22.9 -> 23.7 mm
- net Net-(U6-Pad10): track 40.9 -> 41.5 mm, vias 5 -> 3
- net Net-(U6-Pad7): track 47.5 -> 47.0 mm, vias 5 -> 4
- net /I2C_SDA: track 55.4 -> 55.7 mm, vias 3 -> 0
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
Commit message: small changes to track placement
Connections:
- net /SPI_~CS0 renamed /SPI_~{CS0}
- net /SPI_~CS1 renamed /SPI_~{CS1}
- net /SPI_~HLD~-IO3 renamed /SPI_~{HLD}-IO3
- net /SPI_~WP~-IO2 renamed /SPI_~{WP}-IO2
- net /~LEDM renamed /~{LEDM}
- net /~LEDT renamed /~{LEDT}
Other:
- board text added: "DEUTSCHLAND BUNDESLAENDER STATUS r0.1 Kade Turner"
- board text removed: "DEUTSCHLAND BUNDESLAENDER COVID STATUS Kade Turner"

Commit message: V1 release
Parts:
- U6, U8, U9: value ACSC02-41 -> KCSC02-105
- moved ? 11.6 mm to (114.3, 162.7)
- moved ? 11.6 mm to (114.3, 165.2)
- moved TP1 11.6 mm to (113.5, 162.7)
- moved TP15 11.6 mm to (113.5, 165.2)
- moved ? 2.60 mm to (114.3, 155.1)
- moved TP4 2.60 mm to (113.5, 155.1)
- moved ? 2.50 mm to (114.3, 157.7)
- moved TP5 2.50 mm to (113.5, 157.7)
- moved R5 0.41 mm to (102.2, 112.3)
Connections:
- net Net-(C4-Pad1) renamed /VDDA
- net Net-(C8-Pad1) renamed /VDD3P3_RTC
Routing:
- net /I2C_SCL: track 42.5 -> 63.5 mm
- net /I2C_SDA: track 55.7 -> 68.8 mm, vias 0 -> 2
- net /SEG_IRQ: track 54.6 -> 64.9 mm, vias 0 -> 2
- net /~{LEDT}: track 57.2 -> 61.6 mm
- net /~{LEDM}: track 58.3 -> 62.1 mm
- net /VDD3P3_RTC: track 29.4 -> 26.4 mm
- net Net-(U7-Pad7): track 48.1 -> 50.5 mm
- net Net-(D1-Pad5): track 47.3 -> 49.0 mm
- net Net-(D1-Pad4): track 47.7 -> 49.5 mm
- net VBUS: track 36.9 -> 35.5 mm
- net /USB_N: track 39.9 -> 38.9 mm
- net /USB_P: track 39.6 -> 38.6 mm
- net Net-(C11-Pad2): track 7.88 -> 7.08 mm
- net GND: track 47.8 -> 47.6 mm, vias 76 -> 65

Commit message: Altered silkscreen for V1
Parts:
- removed the ? at (72.0, 154.0)
- removed the ? at (72.0, 151.6)
- added kibuzzard-6108F752: G***, kibuzzard-6108F752, F.Cu at (79.0, 152.8)
