File: hw/DeutschlandLaenderStatus-r0.1/kicad-src/7Segment.kicad_sch (KiCad schematic)
At the start: 5 parts

Commit message: Layout complete
Need to added Map Outline still
Parts:
- added D17: Tausend, LED_SMD:LED_0402_1005Metric, symbol Device:LED_Filled
- added D18: Million, LED_SMD:LED_0402_1005Metric, symbol Device:LED_Filled
- added R10, R12, R13: 10k, Resistor_SMD:R_0402_1005Metric, symbol icebreaker-bitsy-rescue:pkl_R_Small-pkl_device
- added R14, R15: 330, Resistor_SMD:R_0402_1005Metric, symbol Device:R
- U7: renamed from U?; footprint Package_DFN_QFN:TQFN-24-1EP_4x4mm_P0.5mm_EP2.8x2.8mm_PullBack_ThermalVias -> Package_DFN_QFN:TQFN-24-1EP_4x4mm_P0.5mm_EP2.8x2.8mm_PullBack
- gave numbers to parts that had none: 4
Connections:
- net +3V3: now also R10.2, R12.2, R13.2, R14.2, R15.2
- net IRQ: now also R13.1
- net SCL: now also R10.1
- net SDA: now also R12.1
- net at U9.3 (CA), U9.8 (CA): now also U7.6 (DIG6); no longer U7.1 (DIG2)
- net at U6.3 (CA), U6.8 (CA): now also U7.5 (DIG5); no longer U7.23 (DIG0)
- net at U8.3 (CA), U8.8 (CA): now also U7.7 (DIG7); no longer U7.24 (DIG1)
- new net: D17.2 (A), R14.1
- new net: D18.2 (A), R15.1
- new net ~LEDM: D18.1 (K)
- new net ~LEDT: D17.1 (K)

Commit message: added artwork
Parts:
- U7: footprint Package_DFN_QFN:TQFN-24-1EP_4x4mm_P0.5mm_EP2.8x2.8mm_PullBack -> kt-footprints:TQFN-24-1EP_4x4mm_P0.5mm_EP2.8x2.8mm_PullBack
Changed lines of the file:
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@@
-(kicad_sch (version 20201015) (generator eeschema)
+(kicad_sch (version 20210126) (generator eeschema)
   (paper "A4")
   (junction (at 51.816 61.468) (diameter 0.9144) (color 0 0 0 0))
@@
   (junction (at 149.098 81.534) (diameter 1.016) (color 0 0 0 0))
   (junction (at 169.672 64.008) (diameter 0.9144) (color 0 0 0 0))
+  (junction (at 169.672 71.628) (diameter 0.9144) (color 0 0 0 0))
   (junction (at 169.672 99.314) (diameter 0.9144) (color 0 0 0 0))
+  (junction (at 169.672 104.648) (diameter 0.9144) (color 0 0 0 0))
   (junction (at 169.672 135.128) (diameter 0.9144) (color 0 0 0 0))
+  (junction (at 169.672 140.208) (diameter 0.9144) (color 0 0 0 0))
   (no_connect (at 113.538 71.628))
   (no_connect (at 113.538 74.168))
@@
     (effects (font (size 1.27 1.27)) (justify right))
   )
+  (symbol (lib_id "power:PWR_FLAG") (at 169.672 71.628 270) (unit 1)
+    (in_bom yes) (on_board yes)
+    (property "Reference" "#FLG0104" (id 0) (at 171.577 71.628 0)
+      (effects (font (size 1.27 1.27)) hide)
+    )
+    (property "Value" "PWR_FLAG" (id 1) (at 173.228 72.136 90)
+      (effects (font (size 1.27 1.27)) (justify left))
+    )
+    (property "Footprint" "" (id 2) (at 169.672 71.628 0)
+      (effects (font (size 1.27 1.27)) hide)
+    )
+    (property "Datasheet" "~" (id 3) (at 169.672 71.628 0)
+      (effects (font (size 1.27 1.27)) hide)
+    )
+    (pin "1")
+  )
+  (symbol (lib_id "power:PWR_FLAG") (at 169.672 104.648 270) (unit 1)
+    (in_bom yes) (on_board yes)
+    (property "Reference" "#FLG0106" (id 0) (at 171.577 104.648 0)
+      (effects (font (size 1.27 1.27)) hide)
+    )
+    (property "Value" "PWR_FLAG" (id 1) (at 173.228 105.156 90)
+      (effects (font (size 1.27 1.27)) (justify left))
+    )
+    (property "Footprint" "" (id 2) (at 169.672 104.648 0)
+      (effects (font (size 1.27 1.27)) hide)
+    )
+    (property "Datasheet" "~" (id 3) (at 169.672 104.648 0)
+      (effects (font (size 1.27 1.27)) hide)
+    )
+    (pin "1")
+  )
+  (symbol (lib_id "power:PWR_FLAG") (at 169.672 140.208 270) (unit 1)
+    (in_bom yes) (on_board yes)
+    (property "Reference" "#FLG0107" (id 0) (at 171.577 140.208 0)
+      (effects (font (size 1.27 1.27)) hide)
+    )
+    (property "Value" "PWR_FLAG" (id 1) (at 173.228 140.716 90)
+      (effects (font (size 1.27 1.27)) (justify left))
+    )
+    (property "Footprint" "" (id 2) (at 169.672 140.208 0)
+      (effects (font (size 1.27 1.27)) hide)
+    )
+    (property "Datasheet" "~" (id 3) (at 169.672 140.208 0)
+      (effects (font (size 1.27 1.27)) hide)
+    )
+    (pin "1")
+  )
   (symbol (lib_id "power:+3V3") (at 57.912 45.974 0) (unit 1)
     (in_bom yes) (on_board yes)
@@
       (effects (font (size 1.27 1.27)) hide)
     )
+    (pin "1")
   )
   (symbol (lib_id "power:+3V3") (at 98.298 33.528 0) (unit 1)
@@
       (effects (font (size 1.27 1.27)) hide)
     )
+    (pin "1")
   )
   (symbol (lib_id "power:+3V3") (at 101.6 144.78 0) (unit 1)
@@
       (effects (font (size 1.27 1.27)) hide)
     )
+    (pin "1")
   )
   (symbol (lib_id "power:GND") (at 95.758 107.188 0) (unit 1)
@@
       (effects (font (size 1.27 1.27)) hide)
     )
+    (pin "1")
   )
   (symbol (lib_id "icebreaker-bitsy-rescue:pkl_R_Small-pkl_device") (at 51.816 53.34 180) (unit 1)
@@
       (effects (font (size 1.27 1.27)) hide)
     )
+    (pin "1")
+    (pin "2")
   )
   (symbol (lib_id "icebreaker-bitsy-rescue:pkl_R_Small-pkl_device") (at 57.912 53.34 180) (unit 1)
@@
       (effects (font (size 1.27 1.27)) hide)
     )
+    (pin "1")
+    (pin "2")
   )
   (symbol (lib_id "icebreaker-bitsy-rescue:pkl_R_Small-pkl_device") (at 63.5 53.34 180) (unit 1)
@@
       (effects (font (size 1.27 1.27)) hide)
     )
+    (pin "1")
+    (pin "2")
   )
   (symbol (lib_id "icebreaker-bitsy-rescue:pkl_R_Small-pkl_device") (at 77.978 45.974 180) (unit 1)
@@
       (effects (font (size 1.27 1.27)) hide)
     )
+    (pin "1")
+    (pin "2")
   )
   (symbol (lib_name "Device:R_3") (lib_id "Device:R") (at 95.25 152.4 90) (unit 1)
@@
       (effects (font (size 1.27 1.27)) (justify left))
     )
+    (pin "1")
+    (pin "2")
   )
   (symbol (lib_name "Device:R_3") (lib_id "Device:R") (at 95.25 162.56 90) (unit 1)
@@
       (effects (font (size 1.27 1.27)) (justify left))
     )
+    (pin "1")
+    (pin "2")
   )
   (symbol (lib_id "Device:LED_Filled") (at 85.09 152.4 0) (unit 1)
@@
       (effects (font (size 1.27 1.27)) hide)
     )
+    (pin "1")
+    (pin "2")
   )
   (symbol (lib_id "Device:LED_Filled") (at 85.09 162.56 0) (unit 1)
@@
       (effects (font (size 1.27 1.27)) hide)
     )
+    (pin "1")
+    (pin "2")
   )
   (symbol (lib_id "Display_Character:KCSA02-105") (at 159.512 53.848 0) (unit 1)
@@
       (effects (font (size 1.27 1.27)) (justify left) hide)
     )
+    (pin "1")
+    (pin "10")
+    (pin "2")
+    (pin "3")
+    (pin "4")
+    (pin "5")
+    (pin "6")
+    (pin "7")
+    (pin "8")
+    (pin "9")
   )
   (symbol (lib_id "Display_Character:KCSA02-105") (at 159.512 89.154 0) (unit 1)
@@
       (effects (font (size 1.27 1.27)) (justify left) hide)
     )
+    (pin "1")
+    (pin "10")
+    (pin "2")
+    (pin "3")
+    (pin "4")
+    (pin "5")
+    (pin "6")
+    (pin "7")
+    (pin "8")
+    (pin "9")
   )
   (symbol (lib_id "Display_Character:KCSA02-105") (at 159.512 124.968 0) (unit 1)
@@
       (effects (font (size 1.27 1.27)) (justify left) hide)
     )
+    (pin "1")
+    (pin "10")
+    (pin "2")
+    (pin "3")
+    (pin "4")
+    (pin "5")
+    (pin "6")
+    (pin "7")
+    (pin "8")
+    (pin "9")
   )
   (symbol (lib_id "Interface_Expansion:AS1115-BQFT") (at 98.298 71.628 0) (unit 1)
@@
     (property "Reference" "U7" (id 0) (at 104.394 39.116 0))
     (property "Value" "AS1115-BQFT" (id 1) (at 106.934 42.164 0))
-    (property "Footprint" "Package_DFN_QFN:TQFN-24-1EP_4x4mm_P0.5mm_EP2.8x2.8mm_PullBack" (id 2) (at 98.298 71.628 0)
+    (property "Footprint" "kt-footprints:TQFN-24-1EP_4x4mm_P0.5mm_EP2.8x2.8mm_PullBack" (id 2) (at 98.298 71.628 0)
       (effects (font (size 1.27 1.27)) hide)
     )
@@
       (effects (font (size 1.27 1.27)) hide)
     )
+    (pin "1")
+    (pin "10")
+    (pin "11")
+    (pin "12")
+    (pin "13")
+    (pin "14")
+    (pin "15")
+    (pin "16")
+    (pin "17")
+    (pin "18")
+    (pin "19")
+    (pin "2")
+    (pin "20")
+    (pin "21")
+    (pin "22")
+    (pin "23")
+    (pin "24")
+    (pin "25")
+    (pin "3")
+    (pin "4")
+    (pin "5")
+    (pin "6")
+    (pin "7")
+    (pin "8")
+    (pin "9")
   )
 )

Commit message: small changes to track placement
Connections:
- net ~LEDM renamed ~{LEDM}
- net ~LEDT renamed ~{LEDT}
Changed lines of the file:
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@@
-(kicad_sch (version 20210126) (generator eeschema)
+(kicad_sch (version 20210621) (generator eeschema)
   (paper "A4")
   (junction (at 51.816 61.468) (diameter 0.9144) (color 0 0 0 0))
@@
     (effects (font (size 1.27 1.27)) (justify right))
   )
-  (hierarchical_label "~LEDT" (shape input) (at 76.2 152.4 180)
+  (hierarchical_label "~{LEDT}" (shape input) (at 76.2 152.4 180)
     (effects (font (size 1.27 1.27)) (justify right))
   )
-  (hierarchical_label "~LEDM" (shape input) (at 76.2 162.56 180)
+  (hierarchical_label "~{LEDM}" (shape input) (at 76.2 162.56 180)
     (effects (font (size 1.27 1.27)) (justify right))
+  )
+  (symbol (lib_id "power:+3V3") (at 57.912 45.974 0) (unit 1)
+    (in_bom yes) (on_board yes)
+    (property "Reference" "#PWR0110" (id 0) (at 57.912 49.784 0)
+      (effects (font (size 1.27 1.27)) hide)
+    )
+    (property "Value" "+3V3" (id 1) (at 57.912 42.164 0))
+    (property "Footprint" "" (id 2) (at 57.912 45.974 0)
+      (effects (font (size 1.27 1.27)) hide)
+    )
+    (property "Datasheet" "" (id 3) (at 57.912 45.974 0)
+      (effects (font (size 1.27 1.27)) hide)
+    )
+    (pin "1")
+  )
+  (symbol (lib_id "power:+3V3") (at 98.298 33.528 0) (unit 1)
+    (in_bom yes) (on_board yes)
+    (property "Reference" "#PWR033" (id 0) (at 98.298 37.338 0)
+      (effects (font (size 1.27 1.27)) hide)
+    )
+    (property "Value" "+3V3" (id 1) (at 98.298 29.718 0))
+    (property "Footprint" "" (id 2) (at 98.298 33.528 0)
+      (effects (font (size 1.27 1.27)) hide)
+    )
+    (property "Datasheet" "" (id 3) (at 98.298 33.528 0)
+      (effects (font (size 1.27 1.27)) hide)
+    )
+    (pin "1")
+  )
+  (symbol (lib_id "power:+3V3") (at 101.6 144.78 0) (unit 1)
+    (in_bom yes) (on_board yes)
+    (property "Reference" "#PWR0111" (id 0) (at 101.6 148.59 0)
+      (effects (font (size 1.27 1.27)) hide)
+    )
+    (property "Value" "+3V3" (id 1) (at 101.6 140.97 0))
+    (property "Footprint" "" (id 2) (at 101.6 144.78 0)
+      (effects (font (size 1.27 1.27)) hide)
+    )
+    (property "Datasheet" "" (id 3) (at 101.6 144.78 0)
+      (effects (font (size 1.27 1.27)) hide)
+    )
+    (pin "1")
   )
   (symbol (lib_id "power:PWR_FLAG") (at 169.672 71.628 270) (unit 1)
@@
       (effects (font (size 1.27 1.27)) hide)
     )
-    (pin "1")
-  )
-  (symbol (lib_id "power:+3V3") (at 57.912 45.974 0) (unit 1)
-    (in_bom yes) (on_board yes)
-    (property "Reference" "#PWR0110" (id 0) (at 57.912 49.784 0)
-      (effects (font (size 1.27 1.27)) hide)
-    )
-    (property "Value" "+3V3" (id 1) (at 57.912 42.164 0))
-    (property "Footprint" "" (id 2) (at 57.912 45.974 0)
-      (effects (font (size 1.27 1.27)) hide)
-    )
-    (property "Datasheet" "" (id 3) (at 57.912 45.974 0)
-      (effects (font (size 1.27 1.27)) hide)
-    )
-    (pin "1")
-  )
-  (symbol (lib_id "power:+3V3") (at 98.298 33.528 0) (unit 1)
-    (in_bom yes) (on_board yes)
-    (property "Reference" "#PWR033" (id 0) (at 98.298 37.338 0)
-      (effects (font (size 1.27 1.27)) hide)
-    )
-    (property "Value" "+3V3" (id 1) (at 98.298 29.718 0))
-    (property "Footprint" "" (id 2) (at 98.298 33.528 0)
-      (effects (font (size 1.27 1.27)) hide)
-    )
-    (property "Datasheet" "" (id 3) (at 98.298 33.528 0)
-      (effects (font (size 1.27 1.27)) hide)
-    )
-    (pin "1")
-  )
-  (symbol (lib_id "power:+3V3") (at 101.6 144.78 0) (unit 1)
-    (in_bom yes) (on_board yes)
-    (property "Reference" "#PWR0111" (id 0) (at 101.6 148.59 0)
-      (effects (font (size 1.27 1.27)) hide)
-    )
-    (property "Value" "+3V3" (id 1) (at 101.6 140.97 0))
-    (property "Footprint" "" (id 2) (at 101.6 144.78 0)
-      (effects (font (size 1.27 1.27)) hide)
-    )
-    (property "Datasheet" "" (id 3) (at 101.6 144.78 0)
-      (effects (font (size 1.27 1.27)) hide)
-    )
